File: LAN.kicad_sch (KiCad schematic)
At the start: 34 parts, among them U1 W5500, U2 MagJack-A70-112-331N126, U7 AG9905LP, Y1 XO32F025000GEHE001

Commit message: chore: add README (#2)
Other:
- title: (none) -> ESP32 PoE
Changed lines of the file:
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@@
 	(generator_version "9.0")
 	(paper "A4")
+	(title_block
+		(title "ESP32 PoE")
+		(rev "v0.1.0")
+	)
 	(bus_alias "LAN"
 		(members "~{SCS}" "SCLK" "MISO" "MOSI" "~{INT}" "~{RST}")

Commit message: feat: redesign to smaller form factor
Parts:
- removed BR1, BR2: ~, ESP32PoE:CDBHM1100L-G, symbol ESP32PoE:CDBHM1100L-G
- removed C15: 100n, Capacitor_SMD:C_0603_1608Metric, symbol Device:C
- removed C16: 22u, Capacitor_SMD:C_0805_2012Metric, symbol HomeLabIO:C
- removed D1: SMAJ58A, ESP32PoE:SMAJ58A, symbol HomeLabIO:SMAJ58A
- removed U7: AG9905LP, ESP32PoE:AG9905LP, symbol ESP32PoE:AG9905LP
- added J6, J7: Conn_02x02_Counter_Clockwise, Hardware Components:Conn_PinHeader_2x02_P2.54mm_Vertical, symbol Hardware Components:Conn_PinHeader_2x02_P2.54mm_Vertical
- C1, C8: footprint Capacitor_SMD:C_0603_1608Metric -> Hardware Components:C_0402_1005Metric; symbol Device:C -> Hardware Components:C_10u_0402_10V; JLCPCB Part # C96446 -> C315248; MPN CL10A106MA8NRNC -> CL05A106MP5NUNC
- C10, C9: footprint Capacitor_SMD:C_0603_1608Metric -> Hardware Components:C_0603_1608Metric; symbol Device:C -> Hardware Components:C_6n8_0603_100V
- C11: footprint Capacitor_SMD:C_0402_1005Metric -> Hardware Components:C_0402_1005Metric; symbol HomeLabIO:C -> Hardware Components:C_100n_0402_16V
- C12: value 22n -> 10n; footprint Capacitor_SMD:C_0603_1608Metric -> Hardware Components:C_0402_1005Metric; symbol Device:C -> Hardware Components:C_10n_0402_25V; JLCPCB Part # C57895 -> C318576; MPN CL10A225KA8NNNC -> CL05B103KA5NNNC
- C13: footprint Capacitor_SMD:C_0603_1608Metric -> Hardware Components:C_0402_1005Metric; symbol Device:C -> Hardware Components:C_10n_0402_25V; JLCPCB Part # C1589 -> C318576; MPN CL10B103KB8NNNC -> CL05B103KA5NNNC
- C14: footprint Capacitor_SMD:C_0603_1608Metric -> Hardware Components:C_0402_1005Metric; symbol Device:C -> Hardware Components:C_4n7_0402_50V; JLCPCB Part # C1705 -> C84705; MPN CL10A475KP8NNNC -> CL05B472KB5NNNC
- C17, C2, C3, C4, C5, C6, C7: footprint Capacitor_SMD:C_0603_1608Metric -> Hardware Components:C_0402_1005Metric; symbol Device:C -> Hardware Components:C_100n_0402_16V; JLCPCB Part # C1591 -> C1525; MPN CL10B104KB8NNNC -> CL05B104KO5NNNC
- C18, C19: footprint Capacitor_SMD:C_0603_1608Metric -> Hardware Components:C_0402_1005Metric; symbol Device:C -> Hardware Components:C_15p_0402_50V; JLCPCB Part # C1644 -> C86285; MPN CL10C150JB8NNNC -> CL05C150JB5NNNC
- R1, R2, R3, R4: footprint Resistor_SMD:R_0603_1608Metric -> Hardware Components:R_0402_1005Metric; symbol Device:R -> Hardware Components:R_49R9_0402_75V; JLCPCB Part # C114625 -> C5936310; MPN RC0603FR-0749R9L -> AC0402FR-7W49R9L
- R5, R7: footprint Resistor_SMD:R_0402_1005Metric -> Hardware Components:R_0402_1005Metric; symbol HomeLabIO:R -> Hardware Components:R_470_0402_50V
- R6: footprint Resistor_SMD:R_0603_1608Metric -> Hardware Components:R_0402_1005Metric; symbol Device:R -> Hardware Components:R_12k4_0402_50V; JLCPCB Part # C137798 -> C138060; MPN RC0603FR-0712K4L -> RC0402FR-0712K4L
- U1: footprint Package_QFP:LQFP-48_7x7mm_P0.5mm -> Hardware Components:LQFP-48_7x7mm_P0.5mm; symbol Interface_Ethernet:W5500 -> Hardware Components:Eth_W5500
- U2: footprint ESP32PoE:TRJG0926HENL -> Hardware Components:RJ45_USAKRO_DGUK111Q334AB2A2DP057; symbol ESP32PoE:LPJG0926HENL -> Hardware Components:RJ45_USAKRO_DGUK111Q334AB2A2DP057
- Y1: footprint ESP32PoE:SMD3225-4P -> Hardware Components:Oscillator_TDK_SMD3225-4P; symbol SqueezeAMPPOE:XO32F025000GEHE001 -> Hardware Components:Oscillator_25MHz_TDK-XO32F025000GEHE001
Connections:
- net +5V: now also J7.4 (Pin_4)
- net GND: now also J7.3 (Pin_3)
- net VINA: now also J6.2 (Pin_2)
- net VINB: now also J6.1 (Pin_1)
- net VINC: now also J7.2 (Pin_2)
- net VIND: now also J7.1 (Pin_1)
- new net RX: J6.4 (Pin_4)
- new net TX: J6.3 (Pin_3)
- no-connect marks 16 -> 15
Other:
- note removed: "PoE"
- moved on the sheet: C1, C4, C5, C6, C7, C8

Commit message: wip: mini form factor
Parts:
- FB1: footprint ESP32PoE:L0805 -> Hardware Components:FB_0805_2012Metric; symbol Device:FerriteBead -> Hardware Components:FB_MH2029-300Y
Changed lines of the file:
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@@
 	)
 	(symbol
-		(lib_id "Device:FerriteBead")
+		(lib_id "Hardware Components:FB_MH2029-300Y")
 		(at 72.39 33.02 90)
 		(unit 1)
@@
 			)
 		)
-		(property "Footprint" "ESP32PoE:L0805"
+		(property "Footprint" "Hardware Components:FB_0805_2012Metric"
 			(at 72.39 34.798 90)
 			(effects
